File: hardware/GPSDO.kicad_sch (KiCad schematic)
At the start: 4 parts, among them J1 IEC_60320_C14_Receptacle, J2 ANTENNA, SW1 Power

Commit message: Revised hardware design
Parts:
- removed J2: ANTENNA, symbol Connector:Conn_Coaxial
Other:
- sheet Loop Controller renamed GPS Receiver
- added sheet DAC (dac.kicad_sch)
- added sheet Front Panel (front.kicad_sch)
- added sheet ocxo (ocxc.kicad_sch)
- sheet GPS Receiver: file controller.kicad_sch -> gps.kicad_sch
- sheet GPS Receiver ports: added ~{INT}; removed GPS_ANT, GPS_GND, INT, SMT_SIG, SMT_WIN, VCO, VREF
- sheet Power Supply ports: added +12V, +3.3V, -12V, Gnd; removed GND
- sheet Processor ports: added RF, VREF_Internal, ~{INT}; removed INT, SMT_SIG, SMT_WIN, VCO, VREF
