File: Hardware/GPSDO.kicad_sch (KiCad schematic)
At the start: 0 parts

Commit message: Updated PCB
Other:
- sheet Logic ports: added none; removed +3.3V
- note added: "Power Supplies for GPSDO +5 @ 1.5A +12 @ 1.5A -12 @ 500mA"
- note removed: "Power Supplies for GPSDO +3.3 @ 500mA +5 @ 1.5A +12 @ 1.5A -12 @ 500mA"
Changed lines of the file:
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@@
 		(company "Dewayne L. Hafenstein")
 	)
-	(text "Power Supplies for GPSDO\n\n+3.3 @ 500mA\n+5 @ 1.5A\n+12 @ 1.5A \n-12 @ 500mA\n"
+	(text "Power Supplies for GPSDO\n\n+5 @ 1.5A\n+12 @ 1.5A \n-12 @ 500mA\n"
 		(exclude_from_sim no)
 		(at 56.388 71.628 0)
@@
 		(pts
 			(xy 260.35 121.92) (xy 260.35 142.24)
-		)
-		(stroke
-			(width 0)
-			(type default)
-		)
-	)
-	(wire
-		(pts
-			(xy 134.62 53.34) (xy 203.2 53.34)
 		)
 		(stroke
@@
 			)
 		)
-		(pin "+3.3V" input
-			(at 203.2 53.34 180)
-			(effects
-				(font
-					(size 1.27 1.27)
-				)
-				(justify left)
-			)
-		)
