File: Hardware/ocxo.kicad_sch (KiCad schematic)
At the start: 24 parts, among them J401 OCXO, J402 OCXO, J403 OCXO Signal, J404 OCXO Voltage, J405 OCXO, U401 ADCMP600, U402 74LVC1G17, X401 IsoTemp 131, X402 Bliley N47/NV47, X403 IsoTemp 143N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

Commit message: Updated PCB
Parts:
- R401: footprint (none) -> Resistor_THT:R_Axial_DIN0207_L6.3mm_D2.5mm_P10.16mm_Horizontal
Changed lines of the file:
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@@
 			)
 		)
-		(property "Footprint" ""
+		(property "Footprint" "Resistor_THT:R_Axial_DIN0207_L6.3mm_D2.5mm_P10.16mm_Horizontal"
 			(at 294.894 162.814 90)
 			(effects

Commit message: updated pcb
Parts:
- removed J401, J402, J405: OCXO, Connector_PinHeader_2.54mm:PinHeader_1x06_P2.54mm_Vertical, symbol Connector:Conn_01x06_Pin
- C401: footprint Capacitor_THT:C_Axial_L3.8mm_D2.6mm_P10.00mm_Horizontal -> Capacitor_THT:C_Axial_L3.8mm_D2.6mm_P7.50mm_Horizontal
- D401, D402, D403, D404: footprint Diode_THT:D_DO-15_P10.16mm_Horizontal -> Diode_SMD:D_SOD-123
- X404: footprint DH_OCXO:C4550-OCXO -> OCXO:C4550-OCXO
- renumbered J403 to J401, J404 to J402, X406 to X405, X405 to X406
Connections:
- net GND: now also X401.5 (Gnd), X402.5 (Gnd), X403.5 (Gnd), X404.2 (Gnd), X405.1 (Gnd), X406.2 (Gnd)
- net VCO: now also X401.1 (Vco), X402.1 (VCO), X403.1 (VCO), X404.3 (EFC), X405.2 (VCO), X406.3 (VCO)
- net VRef: now also X401.2 (Vref), X402.2 (VRef), X403.2 (VRef), X404.4 (VRef), X405.3 (VRef), X406.4 (VRef)
- net at X401.3 (Vs), X402.3 (+V), X403.3 (Vcc): now also J402.2 (Pin_2), X404.5 (Vs), X405.4 (VCC), X406.5 (Vcc)
- net OCXO_Signal: now reaches X404.1 (RF_Out), X405.5 (RF), X406.1 (RF)
- net OCXO_Signal: now also J401.2 (Pin_2)
- net OCXO_Sine_1: now reaches D401.2 (A), D402.1 (K), R401.2, R402.1, R403.2, U401.4 (-)
- net OCXO_Signal_2: now reaches D403.2 (A), D404.1 (K), R406.2, U401.1 (Out), U402.2
- net OCXO_Square: now reaches J401.1 (Pin_1), R406.1
- net OCXO_Sine: now reaches C401.1, J401.3 (Pin_3)
- net OCXO_Sine_2: now reaches R404.1, R405.2, U401.3 (+)
- no-connect marks 3 -> 0
Other:
- note removed: "+V Gnd NC RF VCO VRef"
- note removed: "Polarizing Pin"
- note removed: "Two different boards are used to mount one of the chosen OCXO modules. Different boards are used to simplify the PCB markings and pin connections."
- moved on the sheet: C401, D401, D402, D403, D404, J401, J402, R401, R402, R403, R404, R405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

Commit message: Updated Schematic; Move to SMD
Parts:
- C401: footprint Capacitor_THT:C_Axial_L3.8mm_D2.6mm_P7.50mm_Horizontal -> Capacitor_SMD:C_0603_1608Metric_Pad1.08x0.95mm_HandSolder
- D401, D402, D403, D404: footprint Diode_SMD:D_SOD-123 -> Diode_SMD:D_SOD-323_HandSoldering
- R401, R402, R403, R404, R405, R406: footprint Resistor_THT:R_Axial_DIN0207_L6.3mm_D2.5mm_P10.16mm_Horizontal -> Resistor_SMD:R_0805_2012Metric_Pad1.20x1.40mm_HandSolder
Changed lines of the file:
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@@
 			)
 		)
-		(property "Footprint" "Resistor_THT:R_Axial_DIN0207_L6.3mm_D2.5mm_P10.16mm_Horizontal"
+		(property "Footprint" "Resistor_SMD:R_0805_2012Metric_Pad1.20x1.40mm_HandSolder"
 			(at 275.844 147.066 90)
 			(effects
@@
 			)
 		)
-		(property "Footprint" "Diode_SMD:D_SOD-123"
+		(property "Footprint" "Diode_SMD:D_SOD-323_HandSoldering"
 			(at 318.135 171.45 0)
 			(effects
@@
 			)
 		)
-		(property "Footprint" "Resistor_THT:R_Axial_DIN0207_L6.3mm_D2.5mm_P10.16mm_Horizontal"
+		(property "Footprint" "Resistor_SMD:R_0805_2012Metric_Pad1.20x1.40mm_HandSolder"
 			(at 308.864 129.794 90)
 			(effects
@@
 			)
 		)
-		(property "Footprint" "Diode_SMD:D_SOD-123"
+		(property "Footprint" "Diode_SMD:D_SOD-323_HandSoldering"
 			(at 264.795 152.4 0)
 			(effects
@@
 			)
 		)
-		(property "Footprint" "Resistor_THT:R_Axial_DIN0207_L6.3mm_D2.5mm_P10.16mm_Horizontal"
+		(property "Footprint" "Resistor_SMD:R_0805_2012Metric_Pad1.20x1.40mm_HandSolder"
 			(at 286.004 147.066 90)
 			(effects
@@
 			)
 		)
-		(property "Footprint" "Resistor_THT:R_Axial_DIN0207_L6.3mm_D2.5mm_P10.16mm_Horizontal"
+		(property "Footprint" "Resistor_SMD:R_0805_2012Metric_Pad1.20x1.40mm_HandSolder"
 			(at 261.874 162.814 90)
 			(effects
@@
 			)
 		)
-		(property "Footprint" "Diode_SMD:D_SOD-123"
+		(property "Footprint" "Diode_SMD:D_SOD-323_HandSoldering"
 			(at 264.795 172.72 0)
 			(effects
@@
 			)
 		)
-		(property "Footprint" "Diode_SMD:D_SOD-123"
+		(property "Footprint" "Diode_SMD:D_SOD-323_HandSoldering"
 			(at 318.135 148.59 0)
 			(effects
@@
 			)
 		)
-		(property "Footprint" "Capacitor_THT:C_Axial_L3.8mm_D2.6mm_P7.50mm_Horizontal"
+		(property "Footprint" "Capacitor_SMD:C_0603_1608Metric_Pad1.08x0.95mm_HandSolder"
 			(at 254 163.83 0)
 			(effects
@@
 			)
 		)
-		(property "Footprint" "Resistor_THT:R_Axial_DIN0207_L6.3mm_D2.5mm_P10.16mm_Horizontal"
+		(property "Footprint" "Resistor_SMD:R_0805_2012Metric_Pad1.20x1.40mm_HandSolder"
 			(at 286.004 172.466 90)
 			(effects
@@
 			)
 		)
-		(property "Footprint" "Resistor_THT:R_Axial_DIN0207_L6.3mm_D2.5mm_P10.16mm_Horizontal"
+		(property "Footprint" "Resistor_SMD:R_0805_2012Metric_Pad1.20x1.40mm_HandSolder"
 			(at 275.844 172.466 90)
 			(effects

Commit message: updated pcb
Parts:
- X404: footprint OCXO:C4550-OCXO -> DH_OCXO:VectronC4550-A
Changed lines of the file:
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@@
 			)
 		)
-		(property "Footprint" "OCXO:C4550-OCXO"
+		(property "Footprint" "DH_OCXO:VectronC4550-A"
 			(at 175.26 146.05 0)
 			(effects
