File: Hardware/GPSDO.kicad_pcb (KiCad board)
At the start: 2 copper layers, 276 x 184 mm, 170 parts, among them J201 Line, J202 Earth, J203 Neutral, J204 44472-0453, J301 Ref Divider, J302 GPS ANT, J303 Encoder, J304 Ref Select, J305 Ref Range, J306 GPS Module, J307 LCD, J308 RF 50 Ohm, J309 RF TTL, J310 1PPS TTL, J311 ICSP, J401 OCXO, J402 OCXO, J403 OCXO Signal, J404 OCXO Voltage, J405 OCXO, Q301 2N3904, T201 B82732R2142, T202 14A-56-28, U201 LM7912, U202 LM2574N-3.3, U203 LM2596T-5, U204 LM2596T-12, U301 DAC8571IDGK, U302 NEO-M8M, U303 OP07, U304 OP07, U305 TXS0108EPW, U306 GALI-52, U307 74LVC1G17, U308 74LVC1G17, U309 MCP23017_SO, U310 24AA02-OT, U311 PIC18F27Q43, U401 ADCMP600, U402 74LVC1G17, X401 IsoTemp 131, X402 Bliley N47/NV47, X403 IsoTemp 143N, X404 VECTRON C4550A, X405 IsoTemp 143A, X406 Oscilloquartz 8663

Commit message: updated schematics
Parts:
- removed C301: .5F, Capacitor_THT:DX_5R5VxxxxU_D11.5mm_P5.00mm
- removed D301: 1N5819, Diode_THT:D_DO-41_SOD81_P10.16mm_Horizontal
- removed J302: GPS ANT, Connector_Coaxial:SMA_Amphenol_901-144_Vertical
- removed J303: Encoder, Connector_PinSocket_2.54mm:PinSocket_1x06_P2.54mm_Vertical
- removed J304: Ref Select, Connector_PinSocket_2.54mm:PinSocket_1x03_P2.54mm_Vertical
- removed J305: Ref Range, Connector_PinSocket_2.54mm:PinSocket_1x03_P2.54mm_Vertical
- removed J306: GPS Module, Connector_PinSocket_2.54mm:PinSocket_1x05_P2.54mm_Vertical
- removed J307: LCD, Connector_PinSocket_2.54mm:PinSocket_1x15_P2.54mm_Vertical
- removed J308: RF 50 Ohm, Connector_Coaxial:SMA_Amphenol_901-144_Vertical
- removed R301: 3.3, Resistor_THT:R_Axial_DIN0204_L3.6mm_D1.6mm_P7.62mm_Horizontal
- removed R306: 4.7K, Resistor_THT:R_Axial_DIN0207_L6.3mm_D2.5mm_P10.16mm_Horizontal
- removed the REF** at (306.0, 111.5)
- removed the REF** at (224.5, 122.5)
- removed the REF** at (214.0, 30.0)
- removed the REF** at (98.5, 88.5)
- removed the REF** at (224.5, 111.5)
- removed the REF** at (306.0, 122.5)
- removed the REF** at (224.5, 30.0)
- removed the REF** at (306.0, 30.0)
- removed the REF** at (98.5, 70.0)
- removed the REF** at (224.5, 204.0)
- removed the REF** at (214.0, 204.0)
- removed the REF** at (306.0, 204.0)
- removed the REF** at (40.0, 204.0)
- removed the REF** at (40.0, 30.0)
- removed T202: 14A-56-28, DH_Transformers_Signal:14A-56
- removed U302: NEO-M8M, RF_GPS:ublox_NEO
- removed U305: TXS0108EPW, Package_SO:TSSOP-20_4.4x6.5mm_P0.65mm
- removed U310: 24AA02-OT, Package_TO_SOT_SMD:SOT-23-5
- added C310: 100n, Capacitor_THT:C_Axial_L3.8mm_D2.6mm_P15.00mm_Horizontal, F.Cu at (235.2, 226.9)
- added C314: 100n, Capacitor_THT:C_Axial_L3.8mm_D2.6mm_P15.00mm_Horizontal, F.Cu at (235.2, 231.1)
- added JP201: Tie, Jumper:SolderJumper-2_P1.3mm_Bridged_RoundedPad1.0x1.5mm, F.Cu at (31.1, 40.4)
- added R322: 4.7K, Resistor_THT:R_Axial_DIN0204_L3.6mm_D1.6mm_P7.62mm_Horizontal, F.Cu at (224.5, 201.9)
- added R323: 10K, Resistor_THT:R_Axial_DIN0204_L3.6mm_D1.6mm_P7.62mm_Horizontal, F.Cu at (224.5, 205.0)
- added REF**: MountingHole_4.3mm_M4_Pad, MountingHole:MountingHole_4.3mm_M4_Pad, F.Cu at (30.5, 30.5)
- added T203: FS24-1500, DH_Transformers_Triad:FS-36VA, F.Cu at (56.3, 109.2)
- added U312: PIC18F27Q43, Package_SO:SOIC-28W_7.5x18.7mm_P1.27mm, F.Cu at (263.7, 201.0)
- added U313: FT232RL, Package_SO:SSOP-28_5.3x10.2mm_P0.65mm, F.Cu at (265.4, 238.6)
- D306, D307: value LED -> Red
- D308, D310: value LED -> Green
- D309: value LED -> Yellow
- D311, D312: value LED -> 1N5819; footprint LED_THT:LED_D3.0mm_Horizontal_O3.81mm_Z2.0mm -> Diode_THT:D_DO-41_SOD81_P10.16mm_Horizontal
- D313: value 1N5819 -> Green; footprint Diode_THT:D_DO-41_SOD81_P10.16mm_Horizontal -> LED_THT:LED_D3.0mm_Horizontal_O3.81mm_Z2.0mm
- D314: value 1N5819 -> Red; footprint Diode_THT:D_DO-41_SOD81_P10.16mm_Horizontal -> LED_THT:LED_D3.0mm_Horizontal_O3.81mm_Z2.0mm
- J309: value RF TTL -> RF 50 Ohm
- J310: value 1PPS TTL -> RF TTL
- J311: value ICSP -> 1PPS TTL; footprint Connector_PinSocket_2.54mm:PinSocket_1x05_P2.54mm_Vertical -> Connector_Coaxial:SMA_Amphenol_901-144_Vertical
- R311: value 142 -> 330
- R312, R313: value 150 -> 330
- R314: value 8.55 -> 330
- R316: value 330 -> 142
- R317, R318: value 330 -> 150
- R319: value 330 -> 8.55
- TP301: value Clock -> VRef
- TP302: value VRef -> VCO
- TP303: value VCO -> RF
- TP305: value RF -> Clock
- U311: value PIC18F27Q43 -> 24AA04; footprint Package_SO:SOIC-28W_7.5x18.7mm_P1.27mm -> Package_SO:SOIC-8_5.3x6.2mm_P1.27mm
- moved U308 212.8 mm to (264.1, 185.1), turned to 0 degrees
- moved U307 187.8 mm to (264.1, 181.2), turned to 0 degrees
- moved FB302 181.4 mm to (221.3, 229.4), turned to 0 degrees
- moved R313 174.0 mm to (214.0, 198.7)
- moved TP302 172.9 mm to (253.8, 218.5)
- moved TP303 172.4 mm to (253.8, 222.6)
- moved TP304 172.4 mm to (253.8, 226.6)
- moved TP305 172.4 mm to (253.8, 230.7)
- moved R206 170.4 mm to (169.5, 165.8), turned to 0 degrees
- moved F302 169.8 mm to (213.7, 244.8)
- moved D304 169.8 mm to (215.4, 227.4), turned to 0 degrees
- moved D305 169.7 mm to (215.4, 232.0)
- moved BT301 168.2 mm to (235.2, 201.6)
- moved C214 157.8 mm to (159.8, 177.4), turned to 0 degrees
- moved R209 157.7 mm to (169.5, 175.3), turned to 0 degrees
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Connections:
- net Net-(U309-GPB3) renamed /Logic/LCD_BL
- D311 pad 2: +5V -> Net-(BT301-+)
- D312 pad 1: Net-(D312-K) -> Net-(D311-K)
- D313 pad 2: Net-(BT301-+) -> +5V
- D314 pad 1: Net-(D313-K) -> Net-(D314-K)
- F301 pad 2: Net-(J309-In) -> Net-(J310-In)
- F302 pad 2: Net-(J310-In) -> Net-(J311-In)
- J311 pad 1: /Logic/~{MCLR} -> Net-(J311-In)
- J311 pad 2: +5V -> GND
- R311 pad 1: GND -> Net-(D306-K)
- R311 pad 2: Net-(R310-Pad2) -> /Logic/FAULT_N
- R312 pad 1: Net-(FB301-Pad2) -> Net-(D307-K)
- R312 pad 2: Net-(F301-Pad1) -> /Logic/POWER_N
- R313 pad 1: Net-(FB302-Pad2) -> Net-(D308-K)
- R313 pad 2: Net-(F302-Pad1) -> /Logic/LOCK_N
- R314 pad 1: Net-(R310-Pad2) -> Net-(D309-K)
- R314 pad 2: Net-(J308-In) -> /Logic/HOLDOVER_N
- R315 pad 1: Net-(D306-K) -> Net-(D310-K)
- R315 pad 2: Net-(U309-GPA0) -> /Logic/GPS_N
- R316 pad 1: Net-(D307-K) -> GND
- R316 pad 2: Net-(U309-GPA1) -> Net-(R310-Pad2)
- R317 pad 1: Net-(D308-K) -> Net-(FB301-Pad2)
- R317 pad 2: Net-(U309-GPA2) -> Net-(F301-Pad1)
- R318 pad 1: Net-(D309-K) -> Net-(FB302-Pad2)
- R318 pad 2: Net-(U309-GPA3) -> Net-(F302-Pad1)
- R319 pad 1: Net-(D310-K) -> Net-(R310-Pad2)
- R319 pad 2: Net-(U309-GPA4) -> Net-(J309-In)
- R320 pad 1: Net-(D311-K) -> Net-(D313-K)
- R320 pad 2: Net-(U309-GPA5) -> Net-(U313-CBUS0)
- R321 pad 1: Net-(D312-K) -> Net-(D314-K)
- R321 pad 2: Net-(U309-GPA6) -> Net-(U313-CBUS1)
- TP301 pad 1: Net-(U311-RA6) -> Net-(J304-Pin_2)
- TP302 pad 1: Net-(J304-Pin_2) -> /Logic/VCO
- TP303 pad 1: /Logic/VCO -> /Logic/RF
- TP305 pad 1: /Logic/RF -> Net-(U312-RA6)
- U309 pad 1: Net-(J307-Pin_5) -> /Logic/LCD_RS
- U309 pad 2: Net-(J307-Pin_6) -> /Logic/LCD_RW
- U309 pad 21: Net-(U309-GPA0) -> unconnected-(U309-GPA0-Pad21)
- U309 pad 22: Net-(U309-GPA1) -> unconnected-(U309-GPA1-Pad22)
- U309 pad 23: Net-(U309-GPA2) -> unconnected-(U309-GPA2-Pad23)
- U309 pad 24: Net-(U309-GPA3) -> /Logic/FAULT_N
- U309 pad 25: Net-(U309-GPA4) -> /Logic/POWER_N
- U309 pad 26: Net-(U309-GPA5) -> /Logic/LOCK_N
- U309 pad 27: Net-(U309-GPA6) -> /Logic/HOLDOVER_N
- U309 pad 28: unconnected-(U309-GPA7-Pad28) -> /Logic/GPS_N
- U309 pad 3: Net-(J307-Pin_7) -> /Logic/LCD_E
- U309 pad 5: Net-(J307-Pin_9) -> /Logic/LCD_D4
- U309 pad 6: Net-(J307-Pin_10) -> /Logic/LCD_D5
- U309 pad 7: Net-(J307-Pin_11) -> /Logic/LCD_D6
- U309 pad 8: Net-(J307-Pin_12) -> /Logic/LCD_D7
- U311 pad 1: /Logic/~{MCLR} -> unconnected-(U311-A0-Pad1)
- U311 pad 2: /Logic/VRef_FB -> unconnected-(U311-A1-Pad2)
- U311 pad 3: /Logic/Int_Ref -> unconnected-(U311-A2-Pad3)
- U311 pad 4: unconnected-(U311-RA2-Pad4) -> GND
- U311 pad 5: unconnected-(U311-RA3-Pad5) -> /Logic/SDA
- U311 pad 6: unconnected-(U311-RA4-Pad6) -> /Logic/SCL
- U311 pad 7: unconnected-(U311-RA5-Pad7) -> GND
- U311 pad 8: GND -> Net-(D311-K)
Routing:
- net Net-(U202-VIN): track 281.8 -> 0.00 mm
- net Net-(U201-VI): track 140.2 -> 0.00 mm
- net Net-(J402-Pin_5): track 106.9 -> 0.00 mm
- net Net-(J401-Pin_4): track 100.0 -> 0.00 mm, vias 1 -> 0
- net Net-(J402-Pin_4): track 99.2 -> 0.00 mm
- net Net-(J401-Pin_2): track 97.7 -> 0.00 mm, vias 1 -> 0
- net Net-(J402-Pin_6): track 88.0 -> 0.00 mm
- net +5V: track 85.9 -> 0.00 mm
- net Net-(J402-Pin_1): track 75.1 -> 0.00 mm
- net Net-(J401-Pin_5): track 65.8 -> 0.00 mm
- net Net-(J402-Pin_2): track 61.7 -> 0.00 mm
- net Net-(U204-FB): track 59.2 -> 0.00 mm
- net Net-(J401-Pin_1): track 59.0 -> 0.00 mm
- net GND: track 67.7 -> 13.9 mm
- net Net-(U203-FB): track 53.6 -> 0.00 mm
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Other:
- board size 276 x 184 mm -> 66 x 116.8 mm

Commit message: Updated PCB
Parts:
- removed the C212 at (148.9, 133.7)
- removed the C215 at (148.9, 143.2)
- removed the D202 at (133.9, 179.6)
- removed the L201 at (156.1, 88.8)
- removed the L204 at (141.6, 140.1)
- removed the R204 at (169.5, 159.5)
- removed the R207 at (169.5, 169.0)
- removed the TP205 at (134.1, 155.6)
- removed the U202 at (133.7, 167.8)
- added C305: 0.1, Capacitor_THT:CP_Radial_D5.0mm_P2.50mm, F.Cu at (178.8, 197.6)
- added C306: 0.1, Capacitor_THT:CP_Radial_D5.0mm_P2.50mm, F.Cu at (178.8, 204.1)
- added C307: 0.1, Capacitor_THT:CP_Radial_D5.0mm_P2.50mm, F.Cu at (178.8, 210.7)
- added C308: 0.1, Capacitor_THT:CP_Radial_D5.0mm_P2.50mm, F.Cu at (178.8, 217.2)
- added C310: 4.7, Capacitor_THT:CP_Radial_D5.0mm_P2.50mm, F.Cu at (178.8, 223.8)
- added C311: 47, Capacitor_THT:CP_Radial_D5.0mm_P2.50mm, F.Cu at (178.8, 230.3)
- added C312: 0.1, Capacitor_THT:C_Disc_D3.0mm_W2.0mm_P2.50mm, F.Cu at (189.5, 228.1)
- added J302: Encoder, Connector_PinHeader_2.54mm:PinHeader_1x06_P2.54mm_Vertical, F.Cu at (190.2, 196.6)
- added J303: Ref Select, Connector_PinHeader_2.54mm:PinHeader_1x02_P2.54mm_Vertical, F.Cu at (167.6, 201.2)
- added J304: GPS Module, Connector_PinHeader_2.54mm:PinHeader_1x05_P2.54mm_Vertical, F.Cu at (190.2, 213.9)
- added J305: VCO Range, Connector_PinHeader_2.54mm:PinHeader_1x03_P2.54mm_Vertical, F.Cu at (194.8, 196.6)
- added J306: LCD, Connector_PinHeader_2.54mm:PinHeader_1x14_P2.54mm_Vertical, F.Cu at (185.7, 196.6)
- added J307: Serial, Connector_PinHeader_2.54mm:PinHeader_1x10_P2.54mm_Vertical, F.Cu at (174.8, 202.2)
- added J311: Program, Connector_PinHeader_2.54mm:PinHeader_1x02_P2.54mm_Vertical, F.Cu at (194.8, 206.2)
- added J312: ICSP, Connector_PinHeader_2.54mm:PinHeader_1x05_P2.54mm_Vertical, F.Cu at (194.8, 213.9)
- added J313: USB, Connector_USB:USB_A_Molex_67643_Horizontal, F.Cu at (152.7, 202.2)
- added R401: 470, Resistor_THT:R_Axial_DIN0207_L6.3mm_D2.5mm_P10.16mm_Horizontal, F.Cu at (152.0, 123.0)
- added REF**: MountingHole_4.3mm_M4_Pad, MountingHole:MountingHole_4.3mm_M4_Pad, F.Cu at (223.5, 172.7)
- added REF**: MountingHole_4.3mm_M4_Pad, MountingHole:MountingHole_4.3mm_M4_Pad, F.Cu at (30.5, 172.7)
- added REF**: Heatsink_AAVID_Extruded_531002B00000G_34.9x12.7mm_H25.4mm, Heatsink:Heatsink_AAVID_Extruded_531002B00000G_34.9x12.7mm_H25.4mm, F.Cu at (93.5, 126.5)
- added REF**: MountingHole_4.3mm_M4_Pad, MountingHole:MountingHole_4.3mm_M4_Pad, F.Cu at (224.0, 30.5)
- added REF**: Heatsink_AAVID_Extruded_531002B00000G_34.9x12.7mm_H25.4mm, Heatsink:Heatsink_AAVID_Extruded_531002B00000G_34.9x12.7mm_H25.4mm, F.Cu at (93.5, 89.4)
- added REF**: Heatsink_Stonecold_HS-S01_13.21x6.35mm, Heatsink:Heatsink_Stonecold_HS-S01_13.21x6.35mm, F.Cu at (109.2, 135.1)
- added REF**: MountingHole_4.3mm_M4_Pad, MountingHole:MountingHole_4.3mm_M4_Pad, F.Cu at (127.0, 30.5)
- added U308: MAX232, Package_DIP:DIP-16_W7.62mm_LongPads, F.Cu at (152.4, 129.0)
- J301: footprint Connector_PinSocket_2.54mm:PinSocket_2x02_P2.54mm_Vertical -> Connector_PinHeader_2.54mm:PinHeader_2x02_P2.54mm_Vertical
- RT201, RT202: footprint SamacSys_Parts:N10SP005M -> Capacitor_THT:C_Disc_D14.5mm_W5.0mm_P10.00mm
- TP202: value +19.8 -> +16.9
- TP203: value -19.8 -> -16.9
- moved RT201 151.7 mm to (38.1, 147.3), turned to 180 degrees
- moved X403 146.0 mm to (177.2, 59.2)
- moved X404 140.2 mm to (167.5, 53.7)
- moved R206 118.8 mm to (102.6, 73.9), turned to 90 degrees
- moved RT202 115.5 mm to (73.7, 147.3)
- moved R201 109.9 mm to (59.7, 154.9), turned to 180 degrees
- moved X401 108.8 mm to (177.3, 46.7)
- moved R204 108.7 mm to (106.7, 73.9), turned to 90 degrees
- moved X405 107.4 mm to (186.6, 53.5), turned to -90 degrees
- moved TP202 106.8 mm to (27.9, 154.9)
- moved TP205 104.5 mm to (115.3, 56.9)
- moved C212 103.7 mm to (123.8, 68.6), turned to 180 degrees
- moved C214 101.1 mm to (107.7, 60.5), turned to 180 degrees
- moved R202 94.6 mm to (74.9, 154.9)
- moved R207 91.0 mm to (102.6, 113.5), turned to 90 degrees
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- renumbered C213 to C212, C214 to C213, C216 to C214, C217 to C215, C302 to C301, C303 to C302, C304 to C303, C305 to C304, C310 to C309, C314 to C313, D203 to D202, D204 to D203, D302 to D301, D303 to D302, D304 to D303, D305 to D304, D306 to D305, D307 to D306, D308 to D307, D309 to D308, D310 to D309, D311 to D310, D312 to D311, D313 to D312, D314 to D313, J309 to J308, J310 to J309, J311 to J310, L202 to L201, L203 to L202, L205 to L203, L206 to L204, R205 to R204, R206 to R205, R208 to R206, R209 to R207, R302 to R301, R303 to R302, R304 to R303, R305 to R304, R307 to R305, R308 to R306, R309 to R307, R310 to R308, R316 to R309, R317 to R310, R318 to R311, R319 to R312, R311 to R313, R312 to R314, R313 to R315, R314 to R316, R315 to R317, R320 to R318, R321 to R319, R322 to R320, R323 to R321, T203 to T202, TP206 to TP205, TP207 to TP206, U203 to U202, U204 to U203, U303 to U302, U304 to U303, U306 to U304, U307 to U305, U308 to U306, U309 to U307, U311 to U309, U312 to U310, U313 to U311
Routing:
- net GND: track 13.9 -> 315.7 mm
- net Net-(U202-VIN): track 0.00 -> 192.1 mm
- net Net-(U201-VI): track 0.00 -> 87.6 mm
- net Net-(U203-FB): track 0.00 -> 54.0 mm, vias 0 -> 1
- net Net-(U202-FB): track 0.00 -> 54.0 mm, vias 0 -> 1
- net Net-(D203-K): track 0.00 -> 35.0 mm
- net Net-(D202-K): track 0.00 -> 32.1 mm
- net +5V: track 0.00 -> 28.5 mm
- net +12V: track 0.00 -> 26.3 mm
- net -12V: track 0.00 -> 23.9 mm
- net Net-(D201-Pad3): track 0.00 -> 19.2 mm
- net Net-(D201-Pad2): track 0.00 -> 19.2 mm
- net Earth_Protective: track 136.7 -> 150.2 mm
- net Net-(D201--): track 0.00 -> 10.2 mm
- net Net-(D201-+): track 0.00 -> 10.2 mm
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- added copper zone on B.Cu, net GND
Other:
- board size 66 x 116.8 mm -> 203.2 x 152.4 mm
- board text added: "C201-C206 2200pF safety caps"
- board text added: "RV201-RV203 150V Varistors"

Commit message: updated pcb
Parts:
- removed the J401 at (180.1, 129.7)
- removed the J402 at (184.7, 129.7)
- removed J405: OCXO, Connector_PinHeader_2.54mm:PinHeader_1x06_P2.54mm_Vertical
- removed the REF** at (223.5, 172.7)
- removed the REF** at (30.5, 30.5)
- removed the REF** at (30.5, 172.7)
- removed the REF** at (93.5, 126.5)
- removed the REF** at (224.0, 30.5)
- removed the REF** at (93.5, 89.4)
- removed the REF** at (109.2, 135.1)
- removed the REF** at (127.0, 30.5)
- removed the U307 at (264.8, 222.3)
- added ?: , , F.Cu at (127.0, 173.7)
- added ?: , , F.Cu at (29.5, 29.5)
- added ?: , , F.Cu at (224.5, 29.5)
- added ?: , , F.Cu at (224.5, 173.7)
- added ?: , , F.Cu at (126.7, 29.5)
- added REF**: MountingHole_2.2mm_M2_DIN965_Pad_TopBottom, MountingHole:MountingHole_2.2mm_M2_DIN965_Pad_TopBottom, F.Cu at (93.5, 99.1)
- added REF**: MountingHole_4.3mm_M4_ISO7380_Pad, MountingHole:MountingHole_4.3mm_M4_ISO7380_Pad, F.Cu at (29.5, 173.7)
- added REF**: MountingHole_4.3mm_M4_DIN965_Pad_TopBottom, MountingHole:MountingHole_4.3mm_M4_DIN965_Pad_TopBottom, F.Cu at (137.9, 92.2)
- added REF**: Heatsink_AAVID_Extruded_531002B00000G_34.9x12.7mm_H25.4mm, Heatsink:Heatsink_AAVID_Extruded_531002B00000G_34.9x12.7mm_H25.4mm, F.Cu at (93.5, 126.7)
- added REF**: MountingHole_2.2mm_M2_DIN965_Pad_TopBottom, MountingHole:MountingHole_2.2mm_M2_DIN965_Pad_TopBottom, F.Cu at (93.5, 114.0)
- added REF**: MountingHole_2.2mm_M2_DIN965_Pad_TopBottom, MountingHole:MountingHole_2.2mm_M2_DIN965_Pad_TopBottom, F.Cu at (93.3, 73.7)
- added REF**: Heatsink_AAVID_Extruded_531002B00000G_34.9x12.7mm_H25.4mm, Heatsink:Heatsink_AAVID_Extruded_531002B00000G_34.9x12.7mm_H25.4mm, F.Cu at (93.5, 86.4)
- added REF**: MountingHole_4.3mm_M4_DIN965_Pad_TopBottom, MountingHole:MountingHole_4.3mm_M4_DIN965_Pad_TopBottom, F.Cu at (194.8, 35.3)
- added REF**: MountingHole_2.2mm_M2_DIN965_Pad_TopBottom, MountingHole:MountingHole_2.2mm_M2_DIN965_Pad_TopBottom, F.Cu at (93.5, 139.4)
- added U308: MCP23017_SO, Package_SO:SOIC-28W_7.5x17.9mm_P1.27mm, F.Cu at (212.9, 93.2)
- C301, C303, C304, C309, C313: footprint Capacitor_THT:C_Axial_L3.8mm_D2.6mm_P15.00mm_Horizontal -> Capacitor_THT:C_Axial_L3.8mm_D2.6mm_P7.50mm_Horizontal
- C401: footprint Capacitor_THT:C_Axial_L3.8mm_D2.6mm_P10.00mm_Horizontal -> Capacitor_THT:C_Axial_L3.8mm_D2.6mm_P7.50mm_Horizontal
- D401, D402, D403, D404: footprint Diode_THT:D_DO-15_P10.16mm_Horizontal -> Diode_SMD:D_SOD-123
- J313: footprint Connector_USB:USB_A_Molex_67643_Horizontal -> Connector_PinSocket_2.54mm:PinSocket_1x05_P2.54mm_Vertical
- Q301: footprint Package_TO_SOT_THT:TO-92L_HandSolder -> Package_TO_SOT_THT:TO-92_Inline
- RT201: renamed from RT202; footprint Capacitor_THT:C_Disc_D14.5mm_W5.0mm_P10.00mm -> SamacSys_Parts:N10SP005M
- RT202: renamed from RT201; footprint Capacitor_THT:C_Disc_D14.5mm_W5.0mm_P10.00mm -> SamacSys_Parts:N10SP005M
- U301: value DAC8571IDGK -> DAC8571
- X405: value IsoTemp 143A -> Oscilloquartz 8663; footprint DH_OCXO:ISOTEMP 143A -> DH_OCXO:OQ8663
- X406: value Oscilloquartz 8663 -> IsoTemp 143A; footprint DH_OCXO:OQ8663 -> DH_OCXO:ISOTEMP 143A
- moved U302 166.6 mm to (141.5, 115.1), turned to 90 degrees
- moved J402 163.6 mm to (120.1, 40.4)
- moved R319 157.9 mm to (215.1, 41.1), turned to 180 degrees
- moved R317 151.9 mm to (215.1, 53.1), turned to 180 degrees
- moved R318 148.9 mm to (215.1, 47.0), turned to 180 degrees
- moved J301 148.4 mm to (140.3, 134.4), turned to 90 degrees
- moved U309 147.3 mm to (149.9, 119.6)
- moved R316 142.7 mm to (215.1, 59.2), turned to 180 degrees
- moved Q301 141.9 mm to (197.1, 110.7), turned to 180 degrees
- moved D313 141.4 mm to (219.2, 41.0), turned to 90 degrees
- moved D311 138.7 mm to (158.5, 116.6)
- moved RV301 137.8 mm to (143.0, 109.0), turned to -90 degrees
- moved D312 134.7 mm to (219.2, 47.0), turned to 90 degrees
- moved R315 133.7 mm to (215.1, 65.0), turned to 180 degrees
- moved D310 130.7 mm to (158.5, 121.4)
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- renumbered J403 to J401, J404 to J402, U308 to U307
Connections:
- net Earth_Protective renamed /Power Supply/Earth_Protective
- net Net-(C201-Pad2) renamed /Power Supply/Line_Filter_1
- net Net-(C202-Pad1) renamed /Power Supply/Neutral_Filter_1
- net Net-(C204-Pad1) renamed /Power Supply/Neutral_Filter_2
- net Net-(C204-Pad2) renamed /Power Supply/Line_Filter_2'
- net Net-(D201-+) renamed /Power Supply/Pos_1
- net Net-(D201--) renamed /Power Supply/Neg_1
- net Net-(D201-Pad2) renamed /Power Supply/Secondary_2
- net Net-(D201-Pad3) renamed /Power Supply/Secondary_1
- net Net-(D202-K) renamed /Power Supply/Reg_Pos_5_Out
- net Net-(D203-K) renamed /Power Supply/Reg_Pos_12_Out
- net Net-(D401-A) renamed /OCXO/OCXO_Sine_1
- net Net-(D403-A) renamed /OCXO/OCXO_Signal_2
- net Net-(J201-Pin_1) renamed /Power Supply/Line_Input
- net Net-(J203-Pin_1) renamed /Power Supply/Neutral_Input
- net Net-(J403-Pin_1) renamed /OCXO/OCXO_Square
- net Net-(J403-Pin_3) renamed /OCXO/OCXO_Sine
- net Net-(U201-VI) renamed /Power Supply/Neg_2
- net Net-(U202-FB) renamed /Power Supply/Reg_5_FB
- net Net-(U202-VIN) renamed /Power Supply/Pos_2
- net Net-(U203-FB) renamed /Power Supply/Reg_12_FB
- net Net-(U308-C1+) renamed /Logic/RS232_C1+
- net Net-(U308-C1-) renamed /Logic/RS232_C1-
- net Net-(U308-VS+) renamed /Logic/RS232_VS+
- net Net-(U308-VS-) renamed /Logic/RS232_V-
- net Net-(U401-+) renamed /OCXO/OCXO_Sine_2
- J313 pad 4: unconnected-(J313-ID-Pad4) -> GND
- J401 pad 2: Net-(J403-Pin_2) -> /OCXO/OCXO_Signal
- J402 pad 2: Net-(J404-Pin_2) -> Net-(J402-Pin_2)
- R313 pad 2: /Logic/FAULT_N -> /Logic/LED_Fault
- R314 pad 2: /Logic/POWER_N -> /Logic/LED_Power
- R315 pad 2: /Logic/LOCK_N -> /Logic/LED_LOCK_N
- R316 pad 2: /Logic/HOLDOVER_N -> /Logic/LED_HOLDOVER_N
- R317 pad 2: /Logic/GPS_N -> /Logic/LED_GPS_N
- X401 pad 1: Net-(J401-Pin_5) -> /Logic/VCO
- X401 pad 2: Net-(J401-Pin_6) -> /Logic/VRef
- X401 pad 3: Net-(J401-Pin_1) -> Net-(J402-Pin_2)
- X401 pad 5: Net-(J401-Pin_2) -> GND
- X402 pad 1: Net-(J401-Pin_5) -> /Logic/VCO
- X402 pad 2: Net-(J401-Pin_6) -> /Logic/VRef
- X402 pad 3: Net-(J401-Pin_1) -> Net-(J402-Pin_2)
- X402 pad 5: Net-(J401-Pin_2) -> GND
- X403 pad 1: Net-(J401-Pin_5) -> /Logic/VCO
- X403 pad 2: Net-(J401-Pin_6) -> /Logic/VRef
- X403 pad 3: Net-(J401-Pin_1) -> Net-(J402-Pin_2)
- X403 pad 5: Net-(J401-Pin_2) -> GND
- X404 pad 1: Net-(J402-Pin_4) -> /OCXO/OCXO_Signal
- X404 pad 2: Net-(J402-Pin_2) -> GND
- X404 pad 3: Net-(J402-Pin_5) -> /Logic/VCO
- X404 pad 4: Net-(J402-Pin_6) -> /Logic/VRef
- X404 pad 5: Net-(J402-Pin_1) -> Net-(J402-Pin_2)
- X405 pad 1: Net-(J402-Pin_4) -> GND
- X405 pad 2: Net-(J402-Pin_2) -> /Logic/VCO
- X405 pad 3: Net-(J402-Pin_5) -> /Logic/VRef
- X405 pad 4: Net-(J402-Pin_6) -> Net-(J402-Pin_2)
- X405 pad 5: Net-(J402-Pin_1) -> /OCXO/OCXO_Signal
- X406 pad 1: Net-(J402-Pin_2) -> /OCXO/OCXO_Signal
- X406 pad 2: Net-(J402-Pin_5) -> GND
- X406 pad 3: Net-(J402-Pin_6) -> /Logic/VCO
- X406 pad 4: Net-(J402-Pin_1) -> /Logic/VRef
- X406 pad 5: Net-(J402-Pin_4) -> Net-(J402-Pin_2)
Routing:
- net +5V: track 28.5 -> 612.3 mm, vias 0 -> 5
- net GND: track 315.7 -> 46.5 mm, vias 0 -> 21
- net Net-(U311-CBUS1): track 0.00 -> 154.2 mm, vias 0 -> 1
- net /Logic/VRef: track 0.00 -> 148.6 mm
- net Net-(U311-CBUS0): track 0.00 -> 147.1 mm, vias 0 -> 1
- net /Logic/VCO: track 0.00 -> 105.5 mm
- net /Logic/SDA: track 0.00 -> 94.6 mm, vias 0 -> 6
- net Net-(J402-Pin_2): track 0.00 -> 93.6 mm, vias 0 -> 1
- net /Logic/SCL: track 0.00 -> 89.4 mm, vias 0 -> 4
- net /OCXO/OCXO_Signal: track 0.00 -> 87.8 mm
- net /OCXO/OCXO_Signal_2: track 0.00 -> 87.2 mm, vias 0 -> 1
- net +12V: track 26.3 -> 109.1 mm
- net /Logic/~{RESET}: track 0.00 -> 77.7 mm, vias 0 -> 4
- net /Logic/1PPS: track 0.00 -> 72.4 mm
- net /Logic/USB_RX: track 0.00 -> 63.4 mm, vias 0 -> 2
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Other:
- outline, holes or cut-outs redrawn
- board text added: "+12V"
- board text added: "+5V"
- board text added: "0.3000 mm"
- board text added: "0.5000 mm / 0.1500 mm"
- board text added: "1.6000 mm"
- board text added: "2"
- board text added: "203.2500 mm x 152.4500 mm"
- board text added: "BOARD CHARACTERISTICS"
- board text added: "Board Thickness:"
- board text added: "Board overall dimensions:"
- board text added: "Castellated pads:"
- board text added: "Copper Finish:"
- board text added: "Copper Layer Count:"
- board text added: "Edge card connectors:"
- board text added: "Fault"
- board text added: "GPS"
- board text added: "Hold"
- board text added: "Impedance Control:"
- board text added: "Lock"
- board text added: "Min hole diameter:"
- board text added: "Min track/spacing:"
- board text added: "No"
- board text added: "None"
- board text added: "PWR"
- board text added: "Plated Board Edge:"

Commit message: Updated Schematic; Move to SMD
Parts:
- removed ? (x5): , 
- removed the REF** at (93.5, 99.1)
- removed the REF** at (29.5, 173.7)
- removed the REF** at (137.9, 92.2)
- removed the REF** at (93.5, 126.7)
- removed the REF** at (93.5, 114.0)
- removed the REF** at (93.3, 73.7)
- removed the REF** at (93.5, 86.4)
- removed the REF** at (194.8, 35.3)
- removed the REF** at (93.5, 139.4)
- removed X404: VECTRON C4550A, DH_OCXO:C4550-OCXO
- added R322: 4.7K, Resistor_SMD:R_0805_2012Metric_Pad1.20x1.40mm_HandSolder, F.Cu at (410.6, 182.0)
- added R323: 4.7K, Resistor_SMD:R_0805_2012Metric_Pad1.20x1.40mm_HandSolder, F.Cu at (410.6, 185.0)
- added REF**: MountingHole_4.3mm_M4_ISO7380_Pad, MountingHole:MountingHole_4.3mm_M4_ISO7380_Pad, F.Cu at (152.4, 127.1)
- added REF**: MountingHole_4.3mm_M4_ISO7380_Pad, MountingHole:MountingHole_4.3mm_M4_ISO7380_Pad, F.Cu at (54.9, 127.0)
- added REF**: Heatsink_AAVID_Extruded_531002B02100G_34.9x12.7mm_H25.4mm, Heatsink:Heatsink_AAVID_Extruded_531002B02100G_34.9x12.7mm_H25.4mm, F.Cu at (195.8, 182.6)
- added REF**: Heatsink_AAVID_Extruded_531002B02100G_34.9x12.7mm_H25.4mm, Heatsink:Heatsink_AAVID_Extruded_531002B02100G_34.9x12.7mm_H25.4mm, F.Cu at (195.8, 141.5)
- added REF**: MountingHole_4.3mm_M4_ISO7380_Pad, MountingHole:MountingHole_4.3mm_M4_ISO7380_Pad, F.Cu at (249.9, 54.9)
- added REF**: MountingHole_4.3mm_M4_ISO7380_Pad, MountingHole:MountingHole_4.3mm_M4_ISO7380_Pad, F.Cu at (249.9, 127.0)
- added REF**: MountingHole_4.3mm_M4_ISO7380_Pad, MountingHole:MountingHole_4.3mm_M4_ISO7380_Pad, F.Cu at (54.9, 199.1)
- added REF**: MountingHole_4.3mm_M4_ISO7380_Pad, MountingHole:MountingHole_4.3mm_M4_ISO7380_Pad, F.Cu at (249.9, 199.1)
- added REF**: MountingHole_4.3mm_M4_ISO7380_Pad, MountingHole:MountingHole_4.3mm_M4_ISO7380_Pad, F.Cu at (54.9, 54.9)
- added REF**: MountingHole_4.3mm_M4_ISO7380_Pad, MountingHole:MountingHole_4.3mm_M4_ISO7380_Pad, F.Cu at (152.4, 54.9)
- added REF**: MountingHole_4.3mm_M4_ISO7380_Pad, MountingHole:MountingHole_4.3mm_M4_ISO7380_Pad, F.Cu at (152.4, 199.1)
- C207, C208, C209, C210: footprint Capacitor_THT:CP_Radial_D22.0mm_P10.00mm_SnapIn -> Capacitor_SMD:CP_Elec_18x22
- C211, C212, C213: footprint Capacitor_THT:CP_Radial_D10.0mm_P5.00mm -> Capacitor_SMD:CP_Elec_10x10.5
- C214, C215: value 180 -> 150; footprint Capacitor_THT:CP_Radial_D8.0mm_P5.00mm -> Capacitor_SMD:CP_Elec_10x10
- C301, C303, C304, C309, C401: footprint Capacitor_THT:C_Axial_L3.8mm_D2.6mm_P7.50mm_Horizontal -> Capacitor_SMD:C_0603_1608Metric_Pad1.08x0.95mm_HandSolder
- C302: footprint Capacitor_THT:CP_Radial_D8.0mm_P5.00mm -> Capacitor_SMD:CP_Elec_8x6.9
- C305, C306, C307, C308: footprint Capacitor_THT:CP_Radial_D5.0mm_P2.50mm -> Capacitor_SMD:CP_Elec_4x5.4
- C310: footprint Capacitor_THT:CP_Radial_D5.0mm_P2.50mm -> Capacitor_SMD:CP_Elec_6.3x5.4
- C311: footprint Capacitor_THT:CP_Radial_D5.0mm_P2.50mm -> Capacitor_SMD:CP_Elec_8x6.9
- C312: footprint Capacitor_THT:C_Disc_D3.0mm_W2.0mm_P2.50mm -> Capacitor_SMD:C_0603_1608Metric_Pad1.08x0.95mm_HandSolder
- D202, D203: footprint Diode_THT:D_DO-201AD_P15.24mm_Horizontal -> Diode_SMD:D_SOD-128
- D301, D302, D303, D304: footprint Diode_SMD:D_SMA -> Diode_SMD:D_SMB_Handsoldering
- D310, D311: value 1N5819 -> SS38; footprint Diode_THT:D_DO-41_SOD81_P10.16mm_Horizontal -> Diode_SMD:D_SMB_Handsoldering
- D401, D402, D403, D404: footprint Diode_SMD:D_SOD-123 -> Diode_SMD:D_SOD-323_HandSoldering
- FB301, FB302: footprint Ferrite_THT:LairdTech_28C0236-0JW-10 -> Inductor_SMD:L_0805_2012Metric_Pad1.15x1.40mm_HandSolder
- L301: footprint Inductor_THT:L_Axial_L7.0mm_D3.3mm_P10.16mm_Horizontal_Fastron_MICC -> Inductor_SMD:L_1206_3216Metric_Pad1.42x1.75mm_HandSolder
- R201, R202, R203, R204, R205, R206, R207, R301, R302, R303, R304, R305, R306, R307, R308, R309, R310, R311, R312, R313, R314, R315, R316, R317, R318, R319, R320, R321: footprint Resistor_THT:R_Axial_DIN0204_L3.6mm_D1.6mm_P7.62mm_Horizontal -> Resistor_SMD:R_0805_2012Metric_Pad1.20x1.40mm_HandSolder
- R401, R402, R403, R404, R405, R406: footprint Resistor_THT:R_Axial_DIN0207_L6.3mm_D2.5mm_P10.16mm_Horizontal -> Resistor_SMD:R_0805_2012Metric_Pad1.20x1.40mm_HandSolder
- T201: footprint SamacSys_Parts:B82732R2142B030 -> DH_Transformers_Common_Mode_Chokes:TDK B82732R Series
- U301: value DAC8571 -> DAC8571IDGK
- moved RV301 298.9 mm to (426.2, 204.4), turned to 0 degrees
- moved U302 292.8 mm to (423.8, 192.8), turned to 0 degrees
- moved R206 272.1 mm to (349.7, 187.9), turned to 0 degrees
- moved C309 267.1 mm to (421.7, 177.5)
- moved U301 266.7 mm to (419.5, 164.3)
- moved R204 266.0 mm to (349.7, 182.0), turned to 0 degrees
- moved J302 264.6 mm to (413.5, 149.5), turned to 0 degrees
- moved TP301 264.5 mm to (415.0, 170.8)
- moved U309 263.8 mm to (412.9, 139.4)
- moved R301 263.7 mm to (396.3, 182.0), turned to 0 degrees
- moved J303 263.3 mm to (421.8, 183.6), turned to 0 degrees
- moved R302 259.0 mm to (396.3, 185.0), turned to 0 degrees
- moved R207 258.9 mm to (349.7, 190.8), turned to 0 degrees
- moved J312 253.5 mm to (422.6, 149.5), turned to 0 degrees
- moved R205 253.3 mm to (349.7, 184.9), turned to 0 degrees
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Connections:
- J204 pad 1: /Power Supply/Neutral_Input -> /Power Supply/Line_Input
- J204 pad 2: /Power Supply/Line_Input -> /Power Supply/Neutral_Input
- J204 pad 3: /Power Supply/Neutral_Filter_1 -> /Power Supply/Line_Filter_1
- J204 pad 4: /Power Supply/Line_Filter_1 -> /Power Supply/Neutral_Filter_1
- T201 pad 1: /Power Supply/Line_Filter_1 -> /Power Supply/Neutral_Filter_1
- T201 pad 2: /Power Supply/Neutral_Filter_1 -> /Power Supply/Line_Filter_1
- T201 pad 3: /Power Supply/Neutral_Filter_2 -> /Power Supply/Line_Filter_2'
- T201 pad 4: /Power Supply/Line_Filter_2' -> /Power Supply/Neutral_Filter_2
Routing:
- net +5V: track 612.3 -> 0.00 mm, vias 5 -> 0
- net Net-(U311-CBUS1): track 154.2 -> 0.00 mm, vias 1 -> 0
- net /Logic/VRef: track 148.6 -> 0.00 mm
- net Net-(U311-CBUS0): track 147.1 -> 0.00 mm, vias 1 -> 0
- net +12V: track 109.1 -> 0.00 mm
- net /Logic/VCO: track 105.5 -> 0.00 mm
- net /Logic/SDA: track 94.6 -> 0.00 mm, vias 6 -> 0
- net Net-(J402-Pin_2): track 93.6 -> 0.00 mm, vias 1 -> 0
- net /Logic/SCL: track 89.4 -> 0.00 mm, vias 4 -> 0
- net /OCXO/OCXO_Signal: track 87.8 -> 0.00 mm
- net /OCXO/OCXO_Signal_2: track 87.2 -> 0.00 mm, vias 1 -> 0
- net /Logic/~{RESET}: track 77.7 -> 0.00 mm, vias 4 -> 0
- net /Logic/1PPS: track 72.4 -> 0.00 mm
- net /Power Supply/Earth_Protective: track 146.0 -> 76.9 mm
- net /Logic/USB_RX: track 63.4 -> 0.00 mm, vias 2 -> 0
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Other:
- board size 203.2 x 152.4 mm -> 203.3 x 152.4 mm
- board text added: "0.0118 in"
- board text added: "0.0157 in / 0.0059 in"
- board text added: "0.0630 in"
- board text added: "8.0050 in x 6.0030 in"
- board text removed: "+12V"
- board text removed: "+5V"
- board text removed: "0.3000 mm"
- board text removed: "0.5000 mm / 0.1500 mm"
- board text removed: "1.6000 mm"
- board text removed: "203.2500 mm x 152.4500 mm"
- board text removed: "C201-C206 2200pF safety caps"
- board text removed: "Fault"
- board text removed: "GPS"
- board text removed: "Hold"
- board text removed: "Lock"
- board text removed: "PWR"
- board text removed: "RV201-RV203 150V Varistors"
