File: Hardware/GPSDO.kicad_pcb (KiCad board)
At the start: 2 copper layers, 203.3 x 152.4 mm, 174 parts, among them J201 Line, J202 Earth, J203 Neutral, J204 44472-0453, J302 Encoder, J303 Ref Select, J304 GPS Module, J305 VCO Range, J306 LCD, J307 Serial, J308 RF 50 Ohm, J309 RF TTL, J310 1PPS TTL, J311 Program, J312 ICSP, J313 USB, J314 Ref Select, J401 OCXO Signal, J402 OCXO Voltage, Q301 2N3904, T201 B82732R2142, T202 FS24-1500, U201 LM7912, U202 LM2596T-5, U203 LM2596T-12, U301 DAC8571IDGK, U302 OP07, U303 OP07, U304 GALI-52, U305 74LVC1G17, U306 74LVC1G17, U307 MAX232, U308 MCP23017_SO, U309 24AA04, U310 PIC18F27Q43, U311 FT232RL, U401 ADCMP600, U402 74LVC1G17, X401 IsoTemp 131, X402 Bliley N47/NV47, X403 IsoTemp 143N, X404 VECTRON C4550A, X405 Oscilloquartz 8663, X406 IsoTemp 143A

Commit message: finished pcb drc edits
Parts:
- Q301: footprint Package_TO_SOT_THT:TO-92_Inline -> Package_TO_SOT_THT:TO-92L_HandSolder
- moved ? 6.86 mm to (170.7, 101.6)
- moved TP303 2.59 mm to (219.4, 109.1)
- moved JP201 1.52 mm to (77.2, 194.6)
- moved D306 0.06 mm to (242.7, 94.0)
Routing:
- net /Power Supply/Earth_Protective: track 72.7 -> 138.2 mm
- net /Power Supply/Neutral_Filter_2: track 93.1 -> 134.6 mm
- net /Power Supply/Pos_2: track 153.0 -> 186.1 mm
- net +12V: track 356.7 -> 381.6 mm
- net +5V: track 773.9 -> 796.4 mm, vias 24 -> 21
- net GND: track 465.4 -> 479.7 mm, vias 46 -> 56
- net -12V: track 225.8 -> 216.8 mm
- net /Logic/Int_Ref: track 66.4 -> 71.5 mm
- net Net-(JP301-A): track 8.79 -> 3.98 mm
- net /Logic/VCO: track 265.6 -> 268.2 mm
- net /Logic/VRef: track 196.7 -> 199.3 mm
- net Net-(J305-Pin_1): track 46.3 -> 44.4 mm
- net /Logic/1PPS: track 142.1 -> 143.7 mm
- net /Logic/RF: track 185.9 -> 187.5 mm
- net /Logic/GPS_RX: track 75.9 -> 77.3 mm
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Other:
- board size 203.3 x 152.4 mm -> 203.2 x 152.4 mm
